Commit message: spawn_model_limo

File: urdf/limo_four_acker.xacro (robot description, xacro)
@@ -69,25 +69,4 @@
     <origin xyz="${wheelbase/2} ${-track/2} ${wheel_vertical_offset}" rpy="${M_PI} 0 0" />
   </xacro:limo_right_steering_hinge>
-        <link name="main_steering_link">
-            <inertial>
-              <mass value="0.25" />
-              <inertia ixx="0.00525" ixy="0" ixz="0" iyy="0.00035" iyz="0" izz="0.00525" />
-              <origin xyz="0 0 0" />
-            </inertial>
-            <visual>
-                <origin xyz="0 0 0" rpy="0 0 0" />
-                <geometry>
-                  <mesh filename="package://lab1_mobile_ackermann/meshes/steering.dae" scale="1 1 1"/>
-                </geometry>
-            </visual>
-        </link>
-        <joint name="main_steering" type="revolute">
-            <parent link="base_link"/>
-            <child link="main_steering_link"/>
-            <origin xyz="${wheelbase/2} 0.0 ${wheel_vertical_offset * -2.0}" rpy="${M_PI} 0 0" />
-            <axis xyz="0 0 -1" />
-            <limit lower="-0.523598767" upper="0.523598767" effort="1000" velocity="10.0" />
-            <dynamics damping="0.0" friction="0.0"/>
-        </joint>
     <xacro:limo_wheel parent_prefix="base_link" wheel_prefix="rear_left" reflect="1" fixed_on="false">
         <origin xyz="${-wheelbase/2} ${track/2} ${wheel_vertical_offset}" rpy="0 0 0" />
@@ -97,5 +76,5 @@
     </xacro:limo_wheel>
 <xacro:include filename="$(find lab1_mobile_ackermann)/urdf/limo_four_acker.gazebo" />
-    <gazebo>
+<gazebo>
         <plugin name="gazebo_ros_ackermann_drive" filename="libgazebo_ros_ackermann_drive.so">
         <ros>
@@ -216,76 +195,3 @@
     </sensor>
 </gazebo>
-<gazebo reference="laser_link">
-    <sensor name="laser" type="ray">
-      <always_on>true</always_on>
-      <visualize>false</visualize>
-      <update_rate>10</update_rate>
-      <ray>
-        <scan>
-          <horizontal>
-            <samples>120</samples>
-            <resolution>1.000000</resolution>
-            <min_angle>-3.14159</min_angle>
-            <max_angle>3.14159</max_angle>
-          </horizontal>
-        </scan>
-        <range>
-          <min>0.3</min>
-          <max>15.0</max>
-          <resolution>0.015</resolution>
-        </range>
-        <noise>
-          <type>gaussian</type>
-          <mean>0.0</mean>
-          <stddev>0.01</stddev>
-        </noise>
-      </ray>
-      <plugin name="scan" filename="libgazebo_ros_ray_sensor.so">
-        <ros>
-          <remapping>~/out:=scan</remapping>
-        </ros>
-        <output_type>sensor_msgs/LaserScan</output_type>
-        <frame_name>laser_link</frame_name>
-      </plugin>
-    </sensor>
-  </gazebo>
-    <link name="camera_depth_optical_frame"/>
-    <joint name="camera_depth_optical_joint" type="fixed">
-      <origin xyz="0 0 0" rpy="${-M_PI/2} 0 ${-M_PI/2}" />
-      <parent link="depth_camera_link" />
-      <child link="camera_depth_optical_frame" />
-    </joint>
-<gazebo reference="depth_camera_link">
-          <sensor name="sensor_camera" type="depth">
-            <pose>0.0 0.0 0.0 0.0 0.0 0.0</pose>
-            <always_on>1</always_on>
-            <update_rate>10</update_rate>
-            <visualize>1</visualize>
-            <camera name="limo_camera">
-              <image>
-                <format>R8G8B8</format>
-                <width>400</width>
-                <height>400</height>
-              </image>
-              <clip>
-                <near>0.01</near>
-                <far>10.0</far>
-              </clip>
-            </camera>
-            <plugin name="gazebo_ros_depth_camera_sensor" filename="libgazebo_ros_camera.so">
-              <ros>
-                <namespace>/limo</namespace>
-                <argument>limo_camera/image_raw:=limo_camera/image</argument>
-                <argument>limo_camera/image_depth:=limo_camera/depth/camera_image_depth</argument>
-                <argument>limo_camera/camera_info:=limo_camera/camera_info_raw</argument>
-                <argument>limo_camera/camera_info_depth:=limo_camera/camera_info_depth</argument>
-                <argument>limo_camera/points:=limo_camera/camera_points</argument>
-              </ros>
-              <camera_name>depth_camera_link</camera_name>
-              <frame_name>camera_depth_optical_frame</frame_name>
-              <hack_baseline>0.07</hack_baseline>
-              <min_depth>0.001</min_depth>
-            </plugin>
-        </sensor>
-          </gazebo>
 </robot>
