Commit message: update_spawn#2_kraiwich model

File: description/limo_mobile.xacro (robot description, xacro)
@@ -1,86 +1,207 @@
 <?xml version="1.0"?>
-<robot name="limo_mobile" xmlns:xacro="http://ros.org/wiki/xacro">
-<!-- Variables -->
-<xacro:property name="M_PI" value="3.14159"/>
-<!-- Vehicle Geometries -->
-<xacro:property name="base_x_size" value="0.13" />
-<xacro:property name="base_y_size" value="0.12" />
-<xacro:property name="base_z_size" value="0.1" />
-<xacro:property name="wheelbase" value="0.2"/>
-<xacro:property name="track" value="0.13"/>
-<xacro:property name="wheel_vertical_offset" value="-0.10" />
-<xacro:property name="base_mass" value="2.1557"/>
-<!-- Wheel Geometries -->
-<xacro:property name="wheel_length" value="0.001" />
-<xacro:property name="wheel_radius" value="0.045" />
-<!-- Base Footprint LINK -->
-<link name="base_footprint"/>
-<!-- Base Footprint JOINT -->
-<joint name="base_joint" type="fixed">
-    <parent link="base_footprint"/>
-    <child link="base_link"/>
-    <origin xyz="0.0 0.0 0.15" rpy="0 0 0"/>
-</joint>
-<!-- Base link -->
-<link name="base_link">
-    <visual>
-        <origin xyz="0 0 -0.15" rpy="0 0 1.57" />
-        <geometry>
-            <mesh filename="package://lab1_mobile_ackermann/meshes/limo_optimal.dae" scale="1 1 1"/>
-        </geometry>
-    </visual>
-    <collision>
-        <origin xyz="0 0 0" rpy="0 0 0" />
-        <geometry>
-            <box size="${base_x_size} ${base_y_size} ${base_z_size}"/>
-        </geometry>
-    </collision>
-    <inertial>
-        <origin xyz="0.0 0.0 0.0" />
-        <mass value="${base_mass}" />
-        <inertia ixx="0.0043832566666666675" ixy="0" ixz="0"
-                    iyy="0.004832360833333334" iyz="0"
-                    izz="0.005622784166666667" />
-    </inertial>
-</link>
-<!-- Front Left Wheel -->
-<link name="front_left">
-    <inertial>
-        <mass value="0.25" />
-        <inertia ixx="0.00525" ixy="0" ixz="0" iyy="0.00035" iyz="0" izz="0.00525" />
-        <origin xyz="0 0 0" />
-    </inertial>
-    <visual>
-        <origin xyz="0 0 0" rpy="0 0 0" />
-        <geometry>
-            <cylinder length="0.0001" radius="0.0001" />
-        </geometry>
-    </visual>
-</link>
-<joint name="front_left_steering" type="revolute">
-    <parent link="base_link"/>
-    <child link="front_left"/>
-    <xacro:insert_block name="joint_pose"/>
-    <axis xyz="0 0 1" />
-    <limit lower="-0.523598767" upper="0.523598767" effort="1000" velocity="1.0" />
-    <dynamics damping="0.0" friction="2.0"/>
-</joint>
-<link name="front_left_wheel_link">
-    <inertial>
-        <mass value="0.25" />
-        <inertia ixx="0.00525" ixy="0" ixz="0" iyy="0.00035" iyz="0" izz="0.00525" />
-        <origin xyz="0 0 0" />
-    </inertial>
-    <visual>
-        <origin xyz="0 0 0" rpy="0 0 0" />
-        <geometry>
-            <mesh filename="package://lab1_mobile_ackermann/meshes/limo_optimal_wheels.dae" />
-        </geometry>
-    </visual>
-    <collision>
-        <origin xyz="0 ${wheel_length/2} 0" rpy="1.57 0 0" />
-        <geometry>
-            <cylinder length="${wheel_length}" radius="${wheel_radius}" />
-        </geometry>
-    </collision>
-</link>
+<robot xmlns:xacro="http://www.ros.org/wiki/xacro">
+    <!-- Import the inertial macros -->
+    <xacro:include filename="inertial_macros.xacro"/>
+    <!-- COLOR NAME  -->
+    <material name="white">
+        <color rgba="1 1 1 1" />
+    </material>
+    <material name="black">
+        <color rgba="0 0 0 1"/>
+    </material>
+     <material name="blue">
+        <color rgba="0 0 1 1"/>
+    </material>
+    <!-- base link -->
+    <link name="base_link"/>
+    <!-- chassis link -->
+    <joint name="chassis_joint" type="fixed">
+        <origin xyz="0.0 0.0 0.095" rpy="0.0 0.0 0.0"/>
+        <parent link="base_link"/>
+        <child link="chassis"/>
+    </joint>
+    <link name="chassis">
+        <visual name="">
+            <origin xyz="0.0 0.0 0.0" rpy="0.0 0.0 0.0"/>
+            <geometry>
+                <box size="0.20 0.13 0.1"/>
+            </geometry>
+            <material name="white"/>
+        </visual>
+        <collision>
+            <origin xyz="0.0 0.0 0.0" rpy="0.0 0.0 0.0"/>
+            <geometry>
+                <box size="0.20 0.13 0.1"/>
+            </geometry>
+        </collision>
+        <xacro:inertial_box mass="3.0" x="0.13" y="0.2" z="0.1">
+            <origin xyz="0.0 0.0 0.0" rpy="0 0 0"/>
+        </xacro:inertial_box>
+    </link>
+    <gazebo reference="chassis">
+        <material>Gazebo/White</material>
+    </gazebo>
+    <!-- front left wheel -->
+    <link name="front_left_wheel_joint_link">
+        <inertial>
+            <origin xyz="0.0 0.0 0.0" rpy="0.0 0.0 0.0"/>
+            <mass value="0.1"/>
+            <inertia ixx="0.01" ixy="0.0" ixz="0.0" iyy="0.01" iyz="0.0" izz="0.01"/>
+        </inertial>
+    </link>
+    <joint name="front_left_steering_joint" type="revolute">
+        <origin xyz="0.10 0.07 -0.045" rpy="0.0 0.0 0.0"/>
+        <parent link="chassis"/>
+        <child link="front_left_wheel_joint_link"/>
+        <axis xyz="0.0 0.0 1.0"/>
+        <limit lower="-0.7854" upper="0.7854" effort="0.0" velocity="0.0"/>
+        <!-- <hardwareInterface>PositionJointInterface</hardwareInterface> -->
+    </joint>
+    <link name="front_left_wheel_link">
+        <inertial>
+            <origin xyz="0.0 0.0 0.0" rpy="0.0 0.0 0.0"/>
+            <mass value="0.1"/>
+            <inertia ixx="0.01" ixy="0.0" ixz="0.0" iyy="0.01" iyz="0.0" izz="0.01"/>
+        </inertial>
+        <visual name="">
+            <origin xyz="0.0 0.0 0.0" rpy="0.0 0.0 0.0"/>
+            <geometry>
+                <cylinder radius="0.045" length="0.01"/>
+            </geometry>
+            <material name="blue"/>
+        </visual>
+        <collision>
+            <origin xyz="0.0 0.0 0.0" rpy="0.0 0.0 0.0"/>
+            <geometry>
+                <cylinder radius="0.045" length="0.01"/>
+            </geometry>
+        </collision>
+        <xacro:inertial_cylinder mass="0.1" length="0.01" radius="0.045">
+            <origin xyz="0 0 0" rpy="0 0 0"/>
+        </xacro:inertial_cylinder>
+    </link>
+    <joint name="front_left_wheel" type="continuous">
+        <origin xyz="0.0 0.0 0.0" rpy="-1.57 0.0 0.0"/>
+        <parent link="front_left_wheel_joint_link"/>
+        <child link="front_left_wheel_link"/>
+        <axis xyz="0.0 0.0 1.0"/>
+    </joint>
+    <gazebo reference="front_left_wheel_link">
+        <material>Gazebo/Blue</material>
+    </gazebo>
+    <!-- front right wheel -->
+    <link name="front_right_wheel_joint_link">
+        <inertial>
+            <origin xyz="0.0 0.0 0.0" rpy="0.0 0.0 0.0"/>
+            <mass value="0.1"/>
+            <inertia ixx="0.01" ixy="0.0" ixz="0.0" iyy="0.01" iyz="0.0" izz="0.01"/>
+        </inertial>
+    </link>
+    <joint name="front_right_steering_joint" type="revolute">
+        <origin xyz="0.10 -0.07 -0.045" rpy="0.0 0.0 0.0"/>
+        <parent link="chassis"/>
+        <child link="front_right_wheel_joint_link"/>
+        <axis xyz="0.0 0.0 1.0"/>
+        <limit lower="-0.7854" upper="0.7854" effort="0.0" velocity="0.0"/>
+        <!-- <hardwareInterface>PositionJointInterface</hardwareInterface> -->
+    </joint>
+    <link name="front_right_wheel_link">
+        <inertial>
+            <origin xyz="0.0 0.0 0.0" rpy="0.0 0.0 0.0"/>
+            <mass value="0.1"/>
+            <inertia ixx="0.01" ixy="0.0" ixz="0.0" iyy="0.01" iyz="0.0" izz="0.01"/>
+        </inertial>
+        <visual name="">
+            <origin xyz="0.0 0.0 0.0" rpy="0.0 0.0 0.0"/>
+            <geometry>
+                <cylinder radius="0.045" length="0.01"/>
+            </geometry>
+            <material name="blue"/>
+        </visual>
+        <collision>
+            <origin xyz="0.0 0.0 0.0" rpy="0.0 0.0 0.0"/>
+            <geometry>
+                <cylinder radius="0.045" length="0.01"/>
+            </geometry>
+        </collision>
+        <xacro:inertial_cylinder mass="0.1" length="0.01" radius="0.045">
+            <origin xyz="0 0 0" rpy="0 0 0"/>
+        </xacro:inertial_cylinder>
+    </link>
+    <joint name="front_right_wheel" type="continuous">
+        <origin xyz="0.0 0.0 0.0" rpy="-1.57 0.0 0.0"/>
+        <parent link="front_right_wheel_joint_link"/>
+        <child link="front_right_wheel_link"/>
+        <axis xyz="0.0 0.0 1.0"/>
+    </joint>
+    <gazebo reference="front_right_wheel_link">
+        <material>Gazebo/Blue</material>
+    </gazebo>
+    <!-- back left wheel -->
+    <joint name="back_left_wheel" type="continuous">
+        <origin xyz="-0.10 0.07 -0.045" rpy="-1.57 0.0 0.0"/>
+        <parent link="chassis"/>
+        <child link="back_left_wheel_link"/>
+        <axis xyz="0.0 0.0 1.0"/>
+    </joint>
+    <link name="back_left_wheel_link">
+        <inertial>
+            <origin xyz="0.0 0.0 0.0" rpy="0.0 0.0 0.0"/>
+            <mass value="0.1"/>
+            <inertia ixx="0.01" ixy="0.0" ixz="0.0" iyy="0.01" iyz="0.0" izz="0.01"/>
+        </inertial>
+        <visual name="">
+            <origin xyz="0.0 0.0 0.0" rpy="0.0 0.0 0.0"/>
+            <geometry>
+                <cylinder radius="0.045" length="0.01"/>
+            </geometry>
+            <material name="black"/>
+        </visual>
+        <collision>
+            <origin xyz="0.0 0.0 0.0" rpy="0.0 0.0 0.0"/>
+            <geometry>
+                <cylinder radius="0.045" length="0.01"/>
+            </geometry>
+        </collision>
+        <xacro:inertial_cylinder mass="0.1" length="0.01" radius="0.045">
+            <origin xyz="0 0 0" rpy="0 0 0"/>
+        </xacro:inertial_cylinder>
+    </link>
+    <gazebo reference="back_left_wheel_link">
+        <material>Gazebo/Black</material>
+    </gazebo>
+    <!-- back right wheel -->
+    <joint name="back_right_wheel" type="continuous">
+        <origin xyz="-0.10 -0.07 -0.045" rpy="-1.57 0.0 0.0"/>
+        <parent link="chassis"/>
+        <child link="back_right_wheel_link"/>
+        <axis xyz="0.0 0.0 1.0"/>
+        <limit lower="0.0" upper="0.0" effort="0.0" velocity="0.0"/>
+    </joint>
+    <link name="back_right_wheel_link">
+        <inertial>
+            <origin xyz="0.0 0.0 0.0" rpy="0.0 0.0 0.0"/>
+            <mass value="0.1"/>
+            <inertia ixx="0.01" ixy="0.0" ixz="0.0" iyy="0.01" iyz="0.0" izz="0.01"/>
+        </inertial>
+        <visual name="">
+            <origin xyz="0.0 0.0 0.0" rpy="0.0 0.0 0.0"/>
+            <geometry>
+                <cylinder radius="0.045" length="0.01"/>
+            </geometry>
+            <material name="black"/>
+        </visual>
+        <collision>
+            <origin xyz="0.0 0.0 0.0" rpy="0.0 0.0 0.0"/>
+            <geometry>
+                <cylinder radius="0.045" length="0.01"/>
+            </geometry>
+        </collision>
+        <xacro:inertial_cylinder mass="0.1" length="0.01" radius="0.045">
+            <origin xyz="0 0 0" rpy="0 0 0"/>
+        </xacro:inertial_cylinder>
+    </link>
+    <gazebo reference="back_right_wheel_link">
+        <material>Gazebo/Black</material>
+    </gazebo>
+</robot>

Commit message: update_spawn#3

File: description/limo_mobile.xacro (robot description, xacro)
@@ -1,109 +1,95 @@
 <?xml version="1.0"?>
-<robot xmlns:xacro="http://www.ros.org/wiki/xacro">
-    <!-- Import the inertial macros -->
+<robot name="limo" xmlns:xacro="http://ros.org/wiki/xacro">
+    <!-- Import macros -->
     <xacro:include filename="inertial_macros.xacro"/>
-    <!-- COLOR NAME  -->
-    <material name="white">
-        <color rgba="1 1 1 1" />
-    </material>
-    <material name="black">
-        <color rgba="0 0 0 1"/>
-    </material>
-     <material name="blue">
-        <color rgba="0 0 1 1"/>
-    </material>
-    <!-- base link -->
-    <link name="base_link"/>
-    <!-- chassis link -->
-    <joint name="chassis_joint" type="fixed">
-        <origin xyz="0.0 0.0 0.095" rpy="0.0 0.0 0.0"/>
-        <parent link="base_link"/>
-        <child link="chassis"/>
-    </joint>
-    <link name="chassis">
-        <visual name="">
-            <origin xyz="0.0 0.0 0.0" rpy="0.0 0.0 0.0"/>
-            <geometry>
-                <box size="0.20 0.13 0.1"/>
-            </geometry>
-            <material name="white"/>
-        </visual>
-        <collision>
-            <origin xyz="0.0 0.0 0.0" rpy="0.0 0.0 0.0"/>
-            <geometry>
-                <box size="0.20 0.13 0.1"/>
-            </geometry>
-        </collision>
-        <xacro:inertial_box mass="3.0" x="0.13" y="0.2" z="0.1">
-            <origin xyz="0.0 0.0 0.0" rpy="0 0 0"/>
-        </xacro:inertial_box>
-    </link>
-    <gazebo reference="chassis">
-        <material>Gazebo/White</material>
-    </gazebo>
-    <!-- front left wheel -->
-    <link name="front_left_wheel_joint_link">
-        <inertial>
-            <origin xyz="0.0 0.0 0.0" rpy="0.0 0.0 0.0"/>
-            <mass value="0.1"/>
-            <inertia ixx="0.01" ixy="0.0" ixz="0.0" iyy="0.01" iyz="0.0" izz="0.01"/>
-        </inertial>
-    </link>
-    <joint name="front_left_steering_joint" type="revolute">
-        <origin xyz="0.10 0.07 -0.045" rpy="0.0 0.0 0.0"/>
-        <parent link="chassis"/>
-        <child link="front_left_wheel_joint_link"/>
-        <axis xyz="0.0 0.0 1.0"/>
-        <limit lower="-0.7854" upper="0.7854" effort="0.0" velocity="0.0"/>
-        <!-- <hardwareInterface>PositionJointInterface</hardwareInterface> -->
-    </joint>
-    <link name="front_left_wheel_link">
-        <inertial>
-            <origin xyz="0.0 0.0 0.0" rpy="0.0 0.0 0.0"/>
-            <mass value="0.1"/>
-            <inertia ixx="0.01" ixy="0.0" ixz="0.0" iyy="0.01" iyz="0.0" izz="0.01"/>
-        </inertial>
-        <visual name="">
-            <origin xyz="0.0 0.0 0.0" rpy="0.0 0.0 0.0"/>
-            <geometry>
-                <cylinder radius="0.045" length="0.01"/>
-            </geometry>
-            <material name="blue"/>
-        </visual>
-        <collision>
-            <origin xyz="0.0 0.0 0.0" rpy="0.0 0.0 0.0"/>
-            <geometry>
-                <cylinder radius="0.045" length="0.01"/>
-            </geometry>
-        </collision>
-        <xacro:inertial_cylinder mass="0.1" length="0.01" radius="0.045">
+    <!-- Base Footprint Link -->
+        <link name="base_footprint"/>
+    <!-- Chassis -->
+        <!-- Joint -->
+        <joint name="chassis_joint" type="fixed">
+            <origin xyz="0 0 0.15" rpy="0 0 0"/>
+            <parent link="base_footprint"/>
+            <child link="chassis"/>
+        </joint>
+        <!-- Link -->
+        <link name="chassis_link">
+            <visual name="">
+                <origin xyz="0 0 -0.15" rpy="0 0 1.57" />
+                <geometry>
+                    <mesh filename="package://lab1_mobile_ackermann/meshes/limo_optimal.dae" scale="1 1 1"/>
+                </geometry>
+            </visual>
+            <collision>
+                <origin xyz="0 0 0" rpy="0 0 0"/>
+                <geometry>
+                    <box size="0.20 0.13 0.1"/>
+                </geometry>
+            </collision>
+            <xacro:inertial_box mass="2.0" x="0.2" y="0.13" z="0.1">
+                <origin xyz="0 0 0" rpy="0 0 0"/>
+            </xacro:inertial_box>
+        </link>
+    <!-- Front Left Steering -->
+        <!-- Link -->
+        <link name="front_left_steering_link">
+            <inertial>
+                <origin xyz="0 0 0" rpy="0 0 0"/>
+                <mass value="0.1"/>
+                <inertia ixx="0.01" ixy="0.0" ixz="0.0" iyy="0.01" iyz="0.0" izz="0.01"/>
+            </inertial>
+        </link>
+        <!-- Joint -->
+        <joint name="front_left_steering_joint" type="revolute">
+            <origin xyz="0.1 0.07 -0.1" rpy="0 0 0"/>
+            <parent link="chassis_link"/>
+            <child link="front_left_steering_link"/>
+            <axis xyz="0 0 1"/>
+            <limit lower="-0.523598767" upper="0.523598767" effort="1000" velocity="1.0" />
+        </joint>
+    <!-- Front Left Wheel -->
+        <!-- Link -->
+        <link name="front_left_wheel_link">
+            <visual>
+              <origin xyz="0 0 0" rpy="0 0 0"/>
+              <geometry>
+                  <mesh filename="package://lab1_mobile_ackermann/meshes/limo_optimal_wheels.dae" />
+              </geometry>
+            </visual>
+            <collision>
+                <origin xyz="0.0 0.005 0.0" rpy="1.57 0.0 0.0"/>
+                <geometry>
+                    <cylinder radius="0.045" length="0.01"/>
+                </geometry>
+            </collision>
+            <xacro:inertial_cylinder mass="0.25" length="0.01" radius="0.045">
+                <origin xyz="0 0 0" rpy="0 0 0"/>
+            </xacro:inertial_cylinder>
+        </link>
+        <!-- Joint -->
+        <joint name="front_left_wheel_joint" type="continuous">
             <origin xyz="0 0 0" rpy="0 0 0"/>
-        </xacro:inertial_cylinder>
-    </link>
-    <joint name="front_left_wheel" type="continuous">
-        <origin xyz="0.0 0.0 0.0" rpy="-1.57 0.0 0.0"/>
-        <parent link="front_left_wheel_joint_link"/>
-        <child link="front_left_wheel_link"/>
-        <axis xyz="0.0 0.0 1.0"/>
-    </joint>
-    <gazebo reference="front_left_wheel_link">
-        <material>Gazebo/Blue</material>
-    </gazebo>
-    <!-- front right wheel -->
-    <link name="front_right_wheel_joint_link">
-        <inertial>
-            <origin xyz="0.0 0.0 0.0" rpy="0.0 0.0 0.0"/>
-            <mass value="0.1"/>
-            <inertia ixx="0.01" ixy="0.0" ixz="0.0" iyy="0.01" iyz="0.0" izz="0.01"/>
-        </inertial>
-    </link>
-    <joint name="front_right_steering_joint" type="revolute">
-        <origin xyz="0.10 -0.07 -0.045" rpy="0.0 0.0 0.0"/>
-        <parent link="chassis"/>
-        <child link="front_right_wheel_joint_link"/>
-        <axis xyz="0.0 0.0 1.0"/>
-        <limit lower="-0.7854" upper="0.7854" effort="0.0" velocity="0.0"/>
-        <!-- <hardwareInterface>PositionJointInterface</hardwareInterface> -->
-    </joint>
+            <parent link="front_left_steering_link"/>
+            <child link="front_left_wheel_link"/>
+            <axis xyz="0 1 0"/>
+            <limit effort="100.0" velocity="10.0"/>
+        </joint>
+    <!-- Front Right Steering -->
+        <!-- Link -->
+        <link name="front_right_wheel_joint_link">
+            <inertial>
+                <origin xyz="0.0 0.0 0.0" rpy="0.0 0.0 0.0"/>
+                <mass value="0.1"/>
+                <inertia ixx="0.01" ixy="0.0" ixz="0.0" iyy="0.01" iyz="0.0" izz="0.01"/>
+            </inertial>
+        </link>
+        <!-- Joint -->
+        <joint name="front_right_steering_joint" type="revolute">
+            <origin xyz="0.10 -0.07 -0.045" rpy="0.0 0.0 0.0"/>
+            <parent link="chassis"/>
+            <child link="front_right_wheel_joint_link"/>
+            <axis xyz="0.0 0.0 1.0"/>
+            <limit lower="-0.7854" upper="0.7854" effort="0.0" velocity="0.0"/>
+        </joint>
+    <!-- Front Right Wheel -->
     <link name="front_right_wheel_link">
         <inertial>
