Commit message: update_spawn#4_spawn limo in world

File: description/limo.xacro (robot description, xacro)
@@ -3,3 +3,4 @@
     <xacro:include filename="limo_mobile.xacro"/>
     <xacro:include filename="limo_mobile.gazebo"/>
+    <xacro:include filename="limo_controllers.gazebo"/>
 </robot>

File: description/limo_mobile.xacro (robot description, xacro)
@@ -10,5 +10,5 @@
             <origin xyz="0 0 0.15" rpy="0 0 0"/>
             <parent link="base_footprint"/>
-            <child link="chassis"/>
+            <child link="chassis_link"/>
         </joint>
         <!-- Link -->
@@ -17,5 +17,5 @@
                 <origin xyz="0 0 -0.15" rpy="0 0 1.57" />
                 <geometry>
-                    <mesh filename="package://lab1_mobile_ackermann/meshes/limo_optimal.dae" scale="1 1 1"/>
+                    <mesh filename="file://$(find lab1_mobile_ackermann)/meshes/limo_optimal.dae" scale="1 1 1"/>
                 </geometry>
             </visual>
@@ -53,9 +53,9 @@
               <origin xyz="0 0 0" rpy="0 0 0"/>
               <geometry>
-                  <mesh filename="package://lab1_mobile_ackermann/meshes/limo_optimal_wheels.dae" />
+                  <mesh filename="file://$(find lab1_mobile_ackermann)/meshes/limo_optimal_wheels.dae" scale="1 1 1"/>
               </geometry>
             </visual>
             <collision>
-                <origin xyz="0.0 0.005 0.0" rpy="1.57 0.0 0.0"/>
+                <origin xyz="0 0.005 0" rpy="1.57 0 0"/>
                 <geometry>
                     <cylinder radius="0.045" length="0.01"/>
@@ -76,7 +76,7 @@
     <!-- Front Right Steering -->
         <!-- Link -->
-        <link name="front_right_wheel_joint_link">
+        <link name="front_right_steering_link">
             <inertial>
-                <origin xyz="0.0 0.0 0.0" rpy="0.0 0.0 0.0"/>
+                <origin xyz="0 0 0" rpy="0 0 0"/>
                 <mass value="0.1"/>
                 <inertia ixx="0.01" ixy="0.0" ixz="0.0" iyy="0.01" iyz="0.0" izz="0.01"/>
@@ -85,109 +85,90 @@
         <!-- Joint -->
         <joint name="front_right_steering_joint" type="revolute">
-            <origin xyz="0.10 -0.07 -0.045" rpy="0.0 0.0 0.0"/>
-            <parent link="chassis"/>
-            <child link="front_right_wheel_joint_link"/>
-            <axis xyz="0.0 0.0 1.0"/>
-            <limit lower="-0.7854" upper="0.7854" effort="0.0" velocity="0.0"/>
+            <origin xyz="0.1 -0.07 -0.1" rpy="3.14159 0 0"/>
+            <parent link="chassis_link"/>
+            <child link="front_right_steering_link"/>
+            <axis xyz="0 0 -1"/>
+            <limit lower="-0.523598767" upper="0.523598767" effort="1000" velocity="1.0" />
         </joint>
     <!-- Front Right Wheel -->
-    <link name="front_right_wheel_link">
-        <inertial>
-            <origin xyz="0.0 0.0 0.0" rpy="0.0 0.0 0.0"/>
-            <mass value="0.1"/>
-            <inertia ixx="0.01" ixy="0.0" ixz="0.0" iyy="0.01" iyz="0.0" izz="0.01"/>
-        </inertial>
-        <visual name="">
-            <origin xyz="0.0 0.0 0.0" rpy="0.0 0.0 0.0"/>
-            <geometry>
-                <cylinder radius="0.045" length="0.01"/>
-            </geometry>
-            <material name="blue"/>
-        </visual>
-        <collision>
-            <origin xyz="0.0 0.0 0.0" rpy="0.0 0.0 0.0"/>
-            <geometry>
-                <cylinder radius="0.045" length="0.01"/>
-            </geometry>
-        </collision>
-        <xacro:inertial_cylinder mass="0.1" length="0.01" radius="0.045">
+        <!-- Link -->
+        <link name="front_right_wheel_link">
+            <visual>
+              <origin xyz="0 0 0" rpy="0 0 0" />
+              <geometry>
+                  <mesh filename="file://$(find lab1_mobile_ackermann)/meshes/limo_optimal_wheels.dae" scale="1 1 1"/>
+              </geometry>
+            </visual>
+            <collision>
+                <origin xyz="0 0.005 0" rpy="1.57 0 0"/>
+                <geometry>
+                    <cylinder radius="0.045" length="0.01"/>
+                </geometry>
+            </collision>
+            <xacro:inertial_cylinder mass="0.25" length="0.01" radius="0.045">
+                <origin xyz="0 0 0" rpy="0 0 0"/>
+            </xacro:inertial_cylinder>
+        </link>
+        <!-- Joint -->
+        <joint name="front_right_wheel_joint" type="continuous">
             <origin xyz="0 0 0" rpy="0 0 0"/>
-        </xacro:inertial_cylinder>
-    </link>
-    <joint name="front_right_wheel" type="continuous">
-        <origin xyz="0.0 0.0 0.0" rpy="-1.57 0.0 0.0"/>
-        <parent link="front_right_wheel_joint_link"/>
-        <child link="front_right_wheel_link"/>
-        <axis xyz="0.0 0.0 1.0"/>
-    </joint>
-    <gazebo reference="front_right_wheel_link">
-        <material>Gazebo/Blue</material>
-    </gazebo>
-    <!-- back left wheel -->
-    <joint name="back_left_wheel" type="continuous">
-        <origin xyz="-0.10 0.07 -0.045" rpy="-1.57 0.0 0.0"/>
-        <parent link="chassis"/>
-        <child link="back_left_wheel_link"/>
-        <axis xyz="0.0 0.0 1.0"/>
-    </joint>
-    <link name="back_left_wheel_link">
-        <inertial>
-            <origin xyz="0.0 0.0 0.0" rpy="0.0 0.0 0.0"/>
-            <mass value="0.1"/>
-            <inertia ixx="0.01" ixy="0.0" ixz="0.0" iyy="0.01" iyz="0.0" izz="0.01"/>
-        </inertial>
-        <visual name="">
-            <origin xyz="0.0 0.0 0.0" rpy="0.0 0.0 0.0"/>
-            <geometry>
-                <cylinder radius="0.045" length="0.01"/>
-            </geometry>
-            <material name="black"/>
-        </visual>
-        <collision>
-            <origin xyz="0.0 0.0 0.0" rpy="0.0 0.0 0.0"/>
-            <geometry>
-                <cylinder radius="0.045" length="0.01"/>
-            </geometry>
-        </collision>
-        <xacro:inertial_cylinder mass="0.1" length="0.01" radius="0.045">
-            <origin xyz="0 0 0" rpy="0 0 0"/>
-        </xacro:inertial_cylinder>
-    </link>
-    <gazebo reference="back_left_wheel_link">
-        <material>Gazebo/Black</material>
-    </gazebo>
-    <!-- back right wheel -->
-    <joint name="back_right_wheel" type="continuous">
-        <origin xyz="-0.10 -0.07 -0.045" rpy="-1.57 0.0 0.0"/>
-        <parent link="chassis"/>
-        <child link="back_right_wheel_link"/>
-        <axis xyz="0.0 0.0 1.0"/>
-        <limit lower="0.0" upper="0.0" effort="0.0" velocity="0.0"/>
-    </joint>
-    <link name="back_right_wheel_link">
-        <inertial>
-            <origin xyz="0.0 0.0 0.0" rpy="0.0 0.0 0.0"/>
-            <mass value="0.1"/>
-            <inertia ixx="0.01" ixy="0.0" ixz="0.0" iyy="0.01" iyz="0.0" izz="0.01"/>
-        </inertial>
-        <visual name="">
-            <origin xyz="0.0 0.0 0.0" rpy="0.0 0.0 0.0"/>
-            <geometry>
-                <cylinder radius="0.045" length="0.01"/>
-            </geometry>
-            <material name="black"/>
-        </visual>
-        <collision>
-            <origin xyz="0.0 0.0 0.0" rpy="0.0 0.0 0.0"/>
-            <geometry>
-                <cylinder radius="0.045" length="0.01"/>
-            </geometry>
-        </collision>
-        <xacro:inertial_cylinder mass="0.1" length="0.01" radius="0.045">
-            <origin xyz="0 0 0" rpy="0 0 0"/>
-        </xacro:inertial_cylinder>
-    </link>
-    <gazebo reference="back_right_wheel_link">
-        <material>Gazebo/Black</material>
-    </gazebo>
+            <parent link="front_right_steering_link"/>
+            <child link="front_right_wheel_link"/>
+            <axis xyz="0 -1 0"/>
+            <limit effort="100.0" velocity="10.0"/>
+        </joint>
+    <!-- Back Left Wheel -->
+        <!-- Link -->
+        <link name="back_left_wheel_link">
+            <visual>
+              <origin xyz="0 0 0" rpy="0 0 0"/>
+              <geometry>
+                  <mesh filename="file://$(find lab1_mobile_ackermann)/meshes/limo_optimal_wheels.dae" scale="1 1 1"/>
+              </geometry>
+            </visual>
+            <collision>
+                <origin xyz="0 0.005 0" rpy="1.57 0 0"/>
+                <geometry>
+                    <cylinder radius="0.045" length="0.01"/>
+                </geometry>
+            </collision>
+            <xacro:inertial_cylinder mass="0.25" length="0.01" radius="0.045">
+                <origin xyz="0 0 0" rpy="0 0 0"/>
+            </xacro:inertial_cylinder>
+        </link>
+        <!-- Joint -->
+        <joint name="back_left_wheel_joint" type="continuous">
+            <origin xyz="-0.1 0.07 -0.1" rpy="0 0.0 0.0"/>
+            <parent link="chassis_link"/>
+            <child link="back_left_wheel_link"/>
+            <axis xyz="0 1 0"/>
+            <limit effort="100.0" velocity="10.0"/>
+        </joint>
+    <!-- Back Right Wheel -->
+        <!-- Link -->
+        <link name="back_right_wheel_link">
+            <visual>
+              <origin xyz="0 0 0" rpy="0 0 0"/>
+              <geometry>
+                  <mesh filename="file://$(find lab1_mobile_ackermann)/meshes/limo_optimal_wheels.dae" scale="1 1 1"/>
+              </geometry>
+            </visual>
+            <collision>
+                <origin xyz="0 0.005 0" rpy="1.57 0 0"/>
+                <geometry>
+                    <cylinder radius="0.045" length="0.01"/>
+                </geometry>
+            </collision>
+            <xacro:inertial_cylinder mass="0.25" length="0.01" radius="0.045">
+                <origin xyz="0 0 0" rpy="0 0 0"/>
+            </xacro:inertial_cylinder>
+        </link>
+        <!-- Joint -->
+        <joint name="back_right_wheel_joint" type="continuous">
+            <origin xyz="-0.1 -0.07 -0.1" rpy="3.14159 0 0"/>
+            <parent link="chassis_link"/>
+            <child link="back_right_wheel_link"/>
+            <axis xyz="0 -1 0"/>
+            <limit effort="100.0" velocity="10.0"/>
+        </joint>
 </robot>
