Commit message: The robot is back!!!!!!

File: description/gazebo_control.xacro (robot description, xacro)
@@ -12,6 +12,6 @@
         <joint name="front_left_steering_joint">
             <command_interface name="position">
-                <param name="min">-1.5</param>
-                <param name="max">1.5</param>
+                <param name="min">-0.7854</param>
+                <param name="max">0.7854</param>
               </command_interface>
               <state_interface name="position">
@@ -25,6 +25,6 @@
         <joint name="front_right_steering_joint">
             <command_interface name="position">
-                <param name="min">-1.5</param>
-                <param name="max">1.5</param>
+                <param name="min">-0.7854</param>
+                <param name="max">0.7854</param>
               </command_interface>
               <state_interface name="position">

File: description/robot_core.urdf.xacro (robot description, xacro)
@@ -47,5 +47,5 @@
         <origin xyz="0.1 0.07 0"/>
         <axis xyz="0 0 1"/>
-        <limit lower="-1.5" upper="1.5" effort="10.0" velocity="3.0"/>
+        <limit lower="-${pi/4}" upper="${pi/4}" effort="10.0" velocity="3.0"/>
     </joint>
     <joint name="front_left_wheel_joint" type="continuous">
@@ -84,5 +84,5 @@
         <origin xyz="0.1 -0.07 0"/>
         <axis xyz="0 0 1"/>
-        <limit lower="-1.5" upper="1.5" effort="10.0" velocity="3.0"/>
+        <limit lower="-${pi/4}" upper="${pi/4}" effort="10.0" velocity="3.0"/>
     </joint>
     <joint name="front_right_wheel_joint" type="continuous">
@@ -102,5 +102,5 @@
             <origin xyz="0 0 -0.005" rpy="${pi/2} 0 0"/>
             <geometry>
-                <mesh filename="file://$(find ${description_package})/meshes/limo_wheel.dae"/>
+                <mesh filename="file://$(find ${description_package})/meshes/limo_wheel.dae" scale="1 1 1"/>
             </geometry>
         </visual>
@@ -125,5 +125,5 @@
             <origin xyz="0 0 -0.005" rpy="${pi/2} 0 0"/>
             <geometry>
-                <mesh filename="file://$(find ${description_package})/meshes/limo_wheel.dae"/>
+                <mesh filename="file://$(find ${description_package})/meshes/limo_wheel.dae" scale="1 1 1"/>
             </geometry>
         </visual>
@@ -148,5 +148,5 @@
             <origin xyz="0 0 -0.005" rpy="${pi/2} 0 0"/>
             <geometry>
-                <mesh filename="file://$(find ${description_package})/meshes/limo_wheel.dae"/>
+                <mesh filename="file://$(find ${description_package})/meshes/limo_wheel.dae" scale="1 1 1"/>
             </geometry>
         </visual>

Commit message: Oniichan nah ja promm todlong la

File: description/gazebo_control.xacro (robot description, xacro)
@@ -1,4 +1,4 @@
 <?xml version="1.0"?>
-<robot xmlns:xacro="http://www.ros.org/wiki/xacro" name="otto">
+<robot xmlns:xacro="http://www.ros.org/wiki/xacro" name="limo">
     <gazebo>
         <plugin filename="libgazebo_ros2_control.so" name="gazebo_ros2_control">

File: description/robot.urdf.xacro (robot description, xacro)
@@ -1,6 +1,7 @@
 <?xml version="1.0"?>
-<robot xmlns:xacro="http://www.ros.org/wiki/xacro"  name="robot">
+<robot xmlns:xacro="http://www.ros.org/wiki/xacro"  name="limo">
     <xacro:property name="description_package" value="lab1_mobile_ackermann"/>
     <xacro:include filename="robot_core.urdf.xacro"/>
     <xacro:include filename="gazebo_control.xacro"/>
+    <xacro:include filename="gazebo_sensor.xacro"/>
 </robot>

File: description/robot_core.urdf.xacro (robot description, xacro)
@@ -40,4 +40,17 @@
             <origin xyz="0.1 0 0.045" rpy="0 0 0"/>
         </xacro:inertial_box>
+    </link>
+    <!-- IMU -->
+    <joint name="imu_joint" type="fixed">
+        <parent link="base_link"/>
+        <child link="imu_link"/>
+        <origin xyz="-0.1 0 0" rpy="0 0 0"/>
+    </joint>
+    <link name="imu_link">
+    <inertial>
+        <origin xyz="0 0 0" rpy="0 0 0"/>
+        <mass value="0.01"/>
+        <inertia ixx="1e-5" ixy="0" ixz="0" iyy="1e-5" iyz="0" izz="1e-5"/>
+    </inertial>
     </link>
     <!-- FRONT LEFT WHEEL -->
@@ -141,5 +154,5 @@
         <parent link="base_link"/>
         <child link="rear_right_wheel"/>
-        <origin xyz="-0.1 -0.07 0" rpy="${pi/2} 0 0" />
+        <origin xyz="-0.1 -0.07 0" rpy="${pi/2} 0 0"/>
         <axis xyz="0 0 -1"/>
     </joint>
