Commit message: ReStructure#6 - Spawn Limo robot

File: limo_model/description/limo_mobile.xacro (robot description, xacro)
@@ -1,4 +1,4 @@
 <?xml version="1.0"?>
-<robot name="limo" xmlns:xacro="http://ros.org/wiki/xacro">
+<robot name="limo" xmlns:xacro="http://www.ros.org/wiki/xacro">
     <!-- Import macros -->
     <xacro:include filename="inertial_macros.xacro"/>
@@ -17,5 +17,5 @@
                 <origin xyz="0 0 -0.15" rpy="0 0 1.57" />
                 <geometry>
-                    <mesh filename="file://$(find lab1_mobile_ackermann)/meshes/limo_optimal.dae" scale="1 1 1"/>
+                    <mesh filename="file://$(find limo_model)/meshes/limo_optimal.dae" scale="1 1 1"/>
                 </geometry>
             </visual>
@@ -53,5 +53,5 @@
               <origin xyz="0 0 0" rpy="0 0 0"/>
               <geometry>
-                  <mesh filename="file://$(find lab1_mobile_ackermann)/meshes/limo_optimal_wheels.dae" scale="1 1 1"/>
+                  <mesh filename="file://$(find limo_model)/meshes/limo_optimal_wheels.dae" scale="1 1 1"/>
               </geometry>
             </visual>
@@ -97,5 +97,5 @@
               <origin xyz="0 0 0" rpy="0 0 0" />
               <geometry>
-                  <mesh filename="file://$(find lab1_mobile_ackermann)/meshes/limo_optimal_wheels.dae" scale="1 1 1"/>
+                  <mesh filename="file://$(find limo_model)/meshes/limo_optimal_wheels.dae" scale="1 1 1"/>
               </geometry>
             </visual>
@@ -124,5 +124,5 @@
               <origin xyz="0 0 0" rpy="0 0 0"/>
               <geometry>
-                  <mesh filename="file://$(find lab1_mobile_ackermann)/meshes/limo_optimal_wheels.dae" scale="1 1 1"/>
+                  <mesh filename="file://$(find limo_model)/meshes/limo_optimal_wheels.dae" scale="1 1 1"/>
               </geometry>
             </visual>
@@ -151,5 +151,5 @@
               <origin xyz="0 0 0" rpy="0 0 0"/>
               <geometry>
-                  <mesh filename="file://$(find lab1_mobile_ackermann)/meshes/limo_optimal_wheels.dae" scale="1 1 1"/>
+                  <mesh filename="file://$(find limo_model)/meshes/limo_optimal_wheels.dae" scale="1 1 1"/>
               </geometry>
             </visual>
