Commit message: Merge Files

File: limo_model/description/limo.xacro (robot description, xacro)
@@ -4,3 +4,4 @@
     <xacro:include filename="limo_mobile.gazebo"/>
     <xacro:include filename="limo_controllers.gazebo"/>
+    <xacro:include filename="limo_sensor.gazebo"/>
 </robot>

File: limo_model/description/limo_mobile.xacro (robot description, xacro)
@@ -4,10 +4,10 @@
     <xacro:include filename="inertial_macros.xacro"/>
     <!-- Base Footprint Link -->
-        <link name="base_footprint"/>
+        <link name="base_link"/>
     <!-- Chassis -->
         <!-- Joint -->
         <joint name="chassis_joint" type="fixed">
             <origin xyz="0 0 0.15" rpy="0 0 0"/>
-            <parent link="base_footprint"/>
+            <parent link="base_link"/>
             <child link="chassis_link"/>
         </joint>

Commit message: re model

File: limo_model/description/limo.xacro (robot description, xacro)
@@ -4,4 +4,3 @@
     <xacro:include filename="limo_mobile.gazebo"/>
     <xacro:include filename="limo_controllers.gazebo"/>
-    <xacro:include filename="limo_sensor.gazebo"/>
 </robot>

File: limo_model/description/limo_mobile.xacro (robot description, xacro)
@@ -4,10 +4,10 @@
     <xacro:include filename="inertial_macros.xacro"/>
     <!-- Base Footprint Link -->
-        <link name="base_link"/>
+        <link name="base_footprint"/>
     <!-- Chassis -->
         <!-- Joint -->
         <joint name="chassis_joint" type="fixed">
             <origin xyz="0 0 0.15" rpy="0 0 0"/>
-            <parent link="base_link"/>
+            <parent link="base_footprint"/>
             <child link="chassis_link"/>
         </joint>

Commit message: Add IMU

File: limo_model/description/limo.xacro (robot description, xacro)
@@ -4,3 +4,4 @@
     <xacro:include filename="limo_mobile.gazebo"/>
     <xacro:include filename="limo_controllers.gazebo"/>
+    <xacro:include filename="limo_sensor.gazebo"/>
 </robot>

File: limo_model/description/limo_mobile.xacro (robot description, xacro)
@@ -8,5 +8,5 @@
         <!-- Joint -->
         <joint name="chassis_joint" type="fixed">
-            <origin xyz="0 0 0.15" rpy="0 0 0"/>
+            <origin xyz="0.1 0 0.15" rpy="0 0 0"/>
             <parent link="base_footprint"/>
             <child link="chassis_link"/>
@@ -29,4 +29,17 @@
                 <origin xyz="0 0 0" rpy="0 0 0"/>
             </xacro:inertial_box>
+        </link>
+    <!-- IMU -->
+        <joint name="imu_joint" type="fixed">
+            <parent link="chassis_link"/>
+            <child link="imu_link"/>
+            <origin xyz="-0.1 0 -0.1" rpy="0 0 0"/>
+        </joint>
+        <link name="imu_link">
+        <inertial>
+            <origin xyz="0 0 0" rpy="0 0 0"/>
+            <mass value="0.01"/>
+            <inertia ixx="1e-5" ixy="0" ixz="0" iyy="1e-5" iyz="0" izz="1e-5"/>
+        </inertial>
         </link>
     <!-- Front Left Steering -->
